Commit message: modifying xacro

File: lib/duckling_description/urdf/sw_bd0.xacro (robot description, xacro)
@@ -304,5 +304,5 @@
   </collision>
 </link>
-<joint name="neck_pitch_base" type="continuous">
+<joint name="neck_pitch" type="continuous">
   <origin xyz="-0.0013 0.023577 0.394589" rpy="0 0 0"/>
   <parent link="base_link"/>

Commit message: setting up launch files

File: lib/duckling_description/urdf/sw_bd0.xacro (robot description, xacro)
@@ -388,3 +388,56 @@
   <axis xyz="1.0 0.0 -0.0"/>
 </joint>
+<!-- Contact points on URDF -->
+<link name="l_foot_toe">
+  <inertial>
+    <origin xyz="0 0 0" rpy="0 0 0"/>
+    <mass value="0.0"/>
+    <inertia ixx="0.0" iyy="0.0" izz="0.0" ixy="-0.0" iyz="0.0" ixz="0.0"/>
+  </inertial>
+</link>
+<link name="l_foot_heel">
+  <inertial>
+    <origin xyz="0 0 0" rpy="0 0 0"/>
+    <mass value="0.0"/>
+    <inertia ixx="0.0" iyy="0.0" izz="0.0" ixy="-0.0" iyz="0.0" ixz="0.0"/>
+  </inertial>
+</link>
+<joint name="l_toe_ankle" type="fixed">
+  <origin xyz="-0.01 -0.1 -0.07" rpy="0 0 0"/>
+  <parent link="Foot-Left_1_1_1"/>
+  <child link="l_foot_toe"/>
+  <axis xyz="1.0 0.0 0.0"/>
+</joint>
+<joint name="l_heel_ankle" type="fixed">
+  <origin xyz="-0.01 0.05 -0.07" rpy="0 0 0"/>
+  <parent link="Foot-Left_1_1_1"/>
+  <child link="l_foot_heel"/>
+  <axis xyz="1.0 0.0 0.0"/>
+</joint>
+<link name="r_foot_toe">
+  <inertial>
+    <origin xyz="0 0 0" rpy="0 0 0"/>
+    <mass value="0.0"/>
+    <inertia ixx="0.0" iyy="0.0" izz="0.0" ixy="-0.0" iyz="0.0" ixz="0.0"/>
+  </inertial>
+</link>
+<link name="r_foot_heel">
+  <inertial>
+    <origin xyz="0 0 0" rpy="0 0 0"/>
+    <mass value="0.0"/>
+    <inertia ixx="0.0" iyy="0.0" izz="0.0" ixy="-0.0" iyz="0.0" ixz="0.0"/>
+  </inertial>
+</link>
+<joint name="r_toe_ankle" type="fixed">
+  <origin xyz="0.01 -0.1 -0.07" rpy="0 0 0"/>
+  <parent link="Foot-Right_1_1_1"/>
+  <child link="r_foot_toe"/>
+  <axis xyz="1.0 0.0 0.0"/>
+</joint>
+<joint name="r_heel_ankle" type="fixed">
+  <origin xyz="0.01 0.05 -0.07" rpy="0 0 0"/>
+  <parent link="Foot-Right_1_1_1"/>
+  <child link="r_foot_heel"/>
+  <axis xyz="1.0 0.0 0.0"/>
+</joint>
 </robot>
